File: hardware/PowerMeter.sch (KiCad schematic (older format))
At the start: 25 parts, among them Q1 OPTO_NPN, U1 MCP1700, U2 ATMEGA88-PA, X1 CRYSTAL

Commit message: Updated schematic, initial board layout
Parts:
- removed C1: 0.1uF, symbol C
- removed C2: 22pF, symbol C
- removed MOD1: XBEE-00, XBee-00, symbol XBEE-00
- removed U2: ATMEGA88-PA, symbol ATMEGA88-PA
- added C4: 22pF, symbol C
- added C5: 0.1uF, symbol C
- added C9: 10nF, symbol C
- added D1: DIODESCH, symbol DIODESCH
- added H1, H2, H3, H4: HOLE, symbol HOLE
- added J1: AVR-ISP-6, AVR-ISP-6, symbol AVR-ISP-6
- added MOD1: XBEE, XBee, symbol XBEE
- added P1, P10, P2, P3, P4, P5, P6, P7, P9: CONN_1, symbol CONN_1
- added P8: CONN_5, symbol CONN_5
- added U2: ATMEGA88-AU, symbol ATMEGA48/88/168/328-AU
- C3: value 22pF -> 0.1uF
- C6: value 10nF -> 22pF
- renumbered C4 to C1, C5 to C2, D1 to D2, D2 to D3, R5 to R2, R6 to R3, R3 to R4, R4 to R5, R2 to R6
Connections:
- net labels added: MISO, MOSI, RST, SCK
- wire segments 74 -> 95
- no-connect marks 26 -> 20
Other:
- note added: "In System Programming"
- note added: "Mounting holes"
- note added: "Power supply"
- note added: "To do:\ndone: add probe pins\ndone: add extra pins on unused ports\ndone: add diode on batt+"
- note added: "Xbee radio module"
- moved on the sheet: BT1, C1, C2, D2, D3, JP1, JP2, Q1, R1, R2, R3, R4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

Commit message: Updated board layout
Parts:
- removed J1: AVR-ISP-6, AVR-ISP-6, symbol AVR-ISP-6
- added ISP1: AVR-ISP-6, AVR-ISP-6, symbol AVR-ISP-6
Connections:
- net +3V: now also ISP1.2
- net GND: now also JP1.2, JP2.2, ISP1.6; no longer D2.2 (K), D3.2 (K)
- net MISO: now also ISP1.1
- net MOSI: now also ISP1.4
- net RST: now also ISP1.5
- net SCK: now also ISP1.3
- net at R4.2: now also U2.10 ((PCINT22/OC0A/AIN0)_PD6); no longer JP1.2
- net at R5.2: now also U2.11 ((PCINT23/AIN1)_PD7); no longer JP2.2
- net at JP1.1: now also D2.2 (K); no longer U2.10 ((PCINT22/OC0A/AIN0)_PD6)
- net at JP2.1: now also D3.2 (K); no longer U2.11 ((PCINT23/AIN1)_PD7)
Other:
- moved on the sheet: D2, D3, JP1, JP2, R4, R5
