File: hardware/PowerMeter.sch (KiCad schematic (older format))
At the start: 44 parts, among them P1 CONN_1, P10 CONN_1, P11 CONN_1, P12 CONN_1, P2 CONN_1, P3 CONN_1, P4 CONN_1, P5 CONN_1, P6 CONN_1, P7 CONN_1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

Commit message: Adjust a couple of resistor values following initial build
Parts:
- R3: value 670K -> 680K
- R4, R5: value 10K -> 1.8K
Changed lines of the file:
@@
-EESchema Schematic File Version 2  date Sun 09 Oct 2011 15:37:40 BST
+EESchema Schematic File Version 2  date Mon 07 Nov 2011 20:05:48 GMT
 LIBS:dresco
 LIBS:PowerMeter-cache
@@
 Sheet 1 1
 Title ""
-Date "8 oct 2011"
+Date "7 nov 2011"
 Rev "1.0"
 Comp ""
@@
 P 7450 5400
 F 0 "R5" V 7530 5400 50  0000 C CNN
-F 1 "10K" V 7450 5400 50  0000 C CNN
+F 1 "1.8K" V 7450 5400 50  0000 C CNN
 	1    7450 5400
 	0    1    1    0
@@
 P 7450 5050
 F 0 "R4" V 7530 5050 50  0000 C CNN
-F 1 "10K" V 7450 5050 50  0000 C CNN
+F 1 "1.8K" V 7450 5050 50  0000 C CNN
 	1    7450 5050
 	0    1    1    0
@@
 P 7950 4000
 F 0 "R3" V 8030 4000 50  0000 C CNN
-F 1 "670K" V 7950 4000 50  0000 C CNN
+F 1 "680K" V 7950 4000 50  0000 C CNN
 	1    7950 4000
 	0    1    1    0
